File: hardware/V2.2/master.kicad_pcb (KiCad board)
At the start: 4 copper layers, 40 x 40 mm, 125 parts, among them J101 USB-MINI-B-SMD, J102 DRILL, J103 DRILL, J104 DRILL, J105 DRILL, J301 STACK-UP-LOW, J302 STACK-DOWN, J303 STACK-UP-LOW, J304 STACK-DOWN, P201 CON-SENSOR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

Commit message: First test with StepUp script for generating .step files out of kiCAD
Parts:
- D304: footprint SOD-323 -> kicad-libraries:SOD-323
