File: hardware/master_3dfork.kicad_pcb (KiCad board)
At the start: 4 copper layers, 40 x 40 mm, 125 parts, among them J1 USB-MINI-B-SMD, J2 DRILL, J3 DRILL, J4 DRILL, J5 DRILL, J6 STACK-UP-LOW, J7 STACK-DOWN, J8 STACK-UP-LOW, J9 STACK-DOWN, P1 CON-SENSOR, P2 CON-SENSOR, P3 CON-SENSOR, P4 CON-SENSOR, P5 TSTPT_GND, P6 TSTPT_5V, P7 TSTPT_3V3, Q1 2N7002P, SW1 Reset, SW2 Erase, U1 AT91SAM3SXC, U10 CM1293A, U11 CM1293A, U12 LD1117, U13 RT9701XB, U2 82400152, U3 PCA9518PW, U4 CM1293A, U5 CM1293A, U6 CM1293A, U7 CM1293A, U8 CM1293A, U9 CM1293A, X1 16Mhz

Commit message: Update 3d information with changed netlist
Parts:
- C1, C2, C3, C4, C5, C6, C7, C8, C9: footprint kicad-libraries:0402 -> C0402
- C10, C11, C12, C13, C14, C16, C18, C19, C20, C22, C23, C24, C25, C26, C27, C28, C30, C31, C32, C33, C34, C36, C37, C38, FB1, FB2, FB3, FB4: footprint kicad-libraries:0603 -> C0603
- C15, C21, C29, C35, C39, L2: footprint kicad-libraries:0805 -> C0805
- C17: footprint kicad-libraries:3528-21 -> 3528-21
- D1, D2, D3, D4, D5, D6: footprint kicad-libraries:D0603 -> D0603
- D11: footprint kicad-libraries:SOD-128 -> SOD-128
- J1: footprint kicad-libraries:USB-MINI-B-SMD -> USB-MINI-B-SMD
- J2, J3, J4, J5: footprint kicad-libraries:DRILL_NP -> DRILL_NP
- J6, J8: footprint kicad-libraries:BTB08-ACS-TOP -> BTB08-ACS-TOP
- J7, J9: footprint kicad-libraries:BTB08-ACS-BTM -> BTB08-ACS-BTM
- L1: footprint kicad-libraries:WE-CNSW-0603 -> WE-CNSW-0603
- P1, P2, P3, P4: footprint kicad-libraries:CON-SENSOR -> CON-SENSOR
- P5, P6, P7: footprint kicad-libraries:TSTPT -> TSTPT
- Q1: footprint kicad-libraries:SOT23EBC -> SOT23EBC
- R1, R10, R11, R12, R13, R14, R15, R16, R17, R2, R3, R4, R6, R8, R9: footprint kicad-libraries:0603 -> R0603
- RP1, RP2, RP3, RP4, RP5, RP6, RP7, RP8, RP9: footprint kicad-libraries:0603X4 -> 0603X4
- SW1, SW2: footprint kicad-libraries:TACT-SWITCH -> TACT-SWITCH
- U1: footprint kicad-libraries:LQFP100 -> LQFP100
- U10, U11, U4, U5, U6, U7, U8, U9: footprint kicad-libraries:SC-74 -> SC-74
- U13: footprint kicad-libraries:SOT23-5 -> SOT23-5
- U2: footprint kicad-libraries:SOT563-SPEC -> SOT563-SPEC
- U3: footprint kicad-libraries:TSSOP20 -> TSSOP20
- X1: footprint kicad-libraries:CRYSTAL_3225 -> CRYSTAL_3225
- moved G*** 0.07 mm to (156.3, 86.3)
Connections:
- J1 pad 4: (no net) -> Net-(J1-Pad4)
- RP2 pad 4: (no net) -> Net-(RP2-Pad4)
- RP2 pad 5: (no net) -> Net-(RP2-Pad5)
- RP3 pad 2: (no net) -> Net-(RP3-Pad2)
- RP3 pad 3: (no net) -> Net-(RP3-Pad3)
- RP3 pad 6: (no net) -> Net-(RP3-Pad6)
- RP3 pad 7: (no net) -> Net-(RP3-Pad7)
- RP5 pad 6: (no net) -> Net-(RP5-Pad6)
- RP5 pad 7: (no net) -> Net-(RP5-Pad7)
- RP8 pad 2: (no net) -> Net-(RP8-Pad2)
- RP8 pad 3: (no net) -> Net-(RP8-Pad3)
- RP8 pad 6: (no net) -> Net-(RP8-Pad6)
- RP8 pad 7: (no net) -> Net-(RP8-Pad7)
- U1 pad 22: (no net) -> Net-(U1-Pad22)
- U1 pad 30: (no net) -> Net-(U1-Pad30)
- U1 pad 46: (no net) -> Net-(U1-Pad46)
- U1 pad 49: (no net) -> Net-(U1-Pad49)
- U1 pad 61: (no net) -> Net-(U1-Pad61)
- U1 pad 71: (no net) -> Net-(U1-Pad71)
- U1 pad 77: (no net) -> Net-(U1-Pad77)
- U10 pad 1: (no net) -> Net-(U10-Pad1)
- U11 pad 1: (no net) -> Net-(U11-Pad1)
- U8 pad 1: (no net) -> Net-(U8-Pad1)
- U9 pad 1: (no net) -> Net-(U9-Pad1)
Other:
- board text added: "Copyright Tinkerforge GmbH 2017. This documentation describes Open Hardware and is licensed under the CERN OHL v. 1.1. You may redistribute and modify this documentation under the terms of the CERN OHL v.1.1. (http://ohwr.org/cernohl). This documentation is distributed WITHOUT ANY EXPRESS OR IMPLIED WARRANTY, INCLUDING OF MERCHANTABILITY, SATISFACTORY QUALITY AND FITNESS FOR A PARTICULAR PURPOSE.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"
- board text removed: "Copyright Tinkerforge GmbH 2011. This documentation describes Open Hardware and is licensed under the CERN OHL v. 1.1. You may redistribute and modify this documentation under the terms of the CERN OHL v.1.1. (http://ohwr.org/cernohl). This documentation is distributed WITHOUT ANY EXPRESS OR IMPLIED WARRANTY, INCLUDING OF MERCHANTABILITY, SATISFACTORY QUALITY AND FITNESS FOR A PARTICULAR PURPOSE.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"
