File: hardware/master_3dfork.kicad_pcb (KiCad board)
At the start: 4 copper layers, 40 x 40 mm, 125 parts, among them J1 USB-MINI-B-SMD, J2 DRILL, J3 DRILL, J4 DRILL, J5 DRILL, J6 STACK-UP-LOW, J7 STACK-DOWN, J8 STACK-UP-LOW, J9 STACK-DOWN, P1 CON-SENSOR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

Commit message: fix clearances
Parts:
- G***: footprint kicad-libraries:Logo_31x31m -> kicad-libraries:Logo_31x31
