File: hardware/master.kicad_pcb (KiCad board)
At the start: 4 copper layers, 40 x 40 mm, 125 parts, among them J1 USB-MINI-B-SMD, J2 DRILL, J3 DRILL, J4 DRILL, J5 DRILL, J6 STACK-UP-LOW, J7 STACK-DOWN, J8 STACK-UP-LOW, J9 STACK-DOWN, P1 CON-SENSOR, P2 CON-SENSOR, P3 CON-SENSOR, P4 CON-SENSOR, P5 TSTPT_GND, P6 TSTPT_5V, P7 TSTPT_3V3, Q1 2N7002P, SW1 Reset, SW2 Erase, U1 AT91SAM3SXC, U10 CM1293A, U11 CM1293A, U12 LD1117, U13 RT9701XB, U2 82400152, U3 PCA9518PW, U4 CM1293A, U5 CM1293A, U6 CM1293A, U7 CM1293A, U8 CM1293A, U9 CM1293A, X1 16Mhz

Commit message: Fix reordered component paths
Parts:
- C1, C2, C3, C4, C5, C6, C7, C8, C9: footprint C0402 -> kicad-libraries:C0402
- C10, C11, C12, C13, C14, C16, C18, C19, C20, C22, C23, C24, C25, C26, C27, C28, C30, C31, C32, C33, C34, C36, C37, C38, FB1, FB2, FB3, FB4: footprint C0603 -> kicad-libraries:C0603
- C15, C21, C29, C35, C39, L2: footprint C0805 -> kicad-libraries:C0805
- C17: footprint 3528-21 -> kicad-libraries:3528-21
- D1, D2, D3, D4, D5, D6: footprint D0603 -> kicad-libraries:D0603
- D11: footprint SOD-128 -> kicad-libraries:SOD-128
- J1: footprint USB-MINI-B-SMD -> kicad-libraries:USB-MINI-B-SMD
- J2, J3, J4, J5: footprint DRILL_NP -> kicad-libraries:DRILL_NP
- J6, J8: footprint BTB08-ACS-TOP -> kicad-libraries:BTB08-ACS-TOP
- J7, J9: footprint BTB08-ACS-BTM -> kicad-libraries:BTB08-ACS-BTM
- L1: footprint WE-CNSW-0603 -> kicad-libraries:WE-CNSW-0603
- P1, P2, P3, P4: footprint CON-SENSOR -> kicad-libraries:CON-SENSOR
- P5, P6, P7: footprint TSTPT -> kicad-libraries:TSTPT
- Q1: footprint SOT23EBC -> kicad-libraries:SOT23EBC
- R1, R10, R11, R12, R13, R14, R15, R16, R17, R2, R3, R4, R6, R8, R9: footprint R0603 -> kicad-libraries:R0603
- RP1, RP2, RP3, RP4, RP5, RP6, RP7, RP8, RP9: footprint 0603X4 -> kicad-libraries:0603X4
- SW1, SW2: footprint TACT-SWITCH -> kicad-libraries:TACT-SWITCH
- U1: footprint LQFP100 -> kicad-libraries:LQFP100
- U10, U11, U4, U5, U6, U7, U8, U9: footprint SC-74 -> kicad-libraries:SC-74
- U13: footprint SOT23-5 -> kicad-libraries:SOT23-5
- U2: footprint SOT563-SPEC -> kicad-libraries:SOT563-SPEC
- U3: footprint TSSOP20 -> kicad-libraries:TSSOP20
- X1: footprint CRYSTAL_3225 -> kicad-libraries:CRYSTAL_3225
