File: hardware/master.kicad_pcb (KiCad board)
At the start: 4 copper layers, 40 x 40 mm, 125 parts, among them J1 USB-MINI-B-SMD, J2 DRILL, J3 DRILL, J4 DRILL, J5 DRILL, J6 STACK-UP-LOW, J7 STACK-DOWN, J8 STACK-UP-LOW, J9 STACK-DOWN, P1 CON-SENSOR, P2 CON-SENSOR, P3 CON-SENSOR, P4 CON-SENSOR, P5 TSTPT_GND, P6 TSTPT_5V, P7 TSTPT_3V3, Q1 2N7002P, SW1 Reset, SW2 Erase, U1 AT91SAM3SXC, U10 CM1293A, U11 CM1293A, U12 LD1117, U13 RT9701XB, U2 82400152, U3 PCA9518PW, U4 CM1293A, U5 CM1293A, U6 CM1293A, U7 CM1293A, U8 CM1293A, U9 CM1293A, X1 16Mhz

Commit message: move V3.1 toplevel
Parts:
- removed C1, C2, C3, C4, C5, C6, C7, C8, C9: DNP, kicad-libraries:C0402
- removed D10, D7, D8, D9: ESD5V0D3B-TP, kicad-libraries:SOD-323
- removed FB2: FB, kicad-libraries:C0603
- removed the Fiducial_Mark at (161.8, 110.1) (x2)
- removed the Fiducial_Mark at (155.8, 76.9)
- removed the Fiducial_Mark at (129.3, 81.4)
- removed the Fiducial_Mark at (135.8, 83.7)
- removed the Fiducial_Mark at (135.3, 112.3)
- removed R1, R2: 100, kicad-libraries:R0603
- removed R14: 1k, kicad-libraries:R0603
- removed RP1, RP2: 100, kicad-libraries:0603X4
- removed U10, U11, U5, U6, U7, U8, U9: CM1293A, kicad-libraries:SC-74
- added C40: DNP, kicad-libraries:C0402F, B.Cu at (148.8, 87.5)
- added C401: 100nF, C0603, F.Cu at (134.1, 82.6)
- added C41: 10uF, kicad-libraries:C0805E, B.Cu at (148.2, 89.0)
- added C42: 100nF, kicad-libraries:C0603F, B.Cu at (148.1, 90.8)
- added C43: 10uF, kicad-libraries:C0805E, B.Cu at (145.0, 93.3)
- added C44: 100nF, kicad-libraries:C0603F, B.Cu at (145.0, 94.8)
- added C45: 10uF, kicad-libraries:C0805E, B.Cu at (148.7, 82.5)
- added C46: 1uF, kicad-libraries:C0603F, B.Cu at (137.6, 79.7)
- added C47: 1uF, kicad-libraries:C0603F, B.Cu at (141.8, 79.9)
- added C48: 2.2uF, kicad-libraries:C0603F, B.Cu at (158.7, 104.6)
- added C49: 2.2uF, kicad-libraries:C0603F, B.Cu at (158.7, 100.4)
- added C50: 2.2uF, kicad-libraries:C0603F, B.Cu at (144.5, 99.0)
- added C51: 2.2uF, kicad-libraries:C0603F, B.Cu at (144.5, 103.2)
- added CP1: 220pF, kicad-libraries:4X0402, F.Cu at (135.1, 102.4)
- added CP2: 220pF, kicad-libraries:4X0402, F.Cu at (151.1, 102.4)
- added CP3: 220pF, kicad-libraries:4X0402, B.Cu at (138.9, 102.4)
- added CP4: 220pF, kicad-libraries:4X0402, B.Cu at (154.9, 102.5)
- added FB101: FB, C0603, B.Cu at (139.7, 80.4)
- added FB102: FB, C0603, B.Cu at (148.5, 74.3)
- added Fiducial_Mark: VAL**, kicad-libraries:Fiducial_Mark, B.Cu at (154.0, 80.0)
- added Fiducial_Mark: VAL**, kicad-libraries:Fiducial_Mark, B.Cu at (126.5, 77.0)
- added Fiducial_Mark: VAL**, kicad-libraries:Fiducial_Mark, B.Cu at (133.5, 99.5)
- added Fiducial_Mark: VAL**, kicad-libraries:Fiducial_Mark, F.Cu at (159.5, 103.0)
- added Fiducial_Mark: VAL**, kicad-libraries:Fiducial_Mark, F.Cu at (131.5, 105.5)
- added Fiducial_Mark: VAL**, kicad-libraries:Fiducial_Mark, F.Cu at (138.0, 73.5)
- added L3: FB, kicad-libraries:R0603F, B.Cu at (157.8, 102.5)
- added L4: FB, kicad-libraries:R0603F, B.Cu at (143.7, 101.0)
- added L5: FB, kicad-libraries:R0603F, B.Cu at (159.4, 102.5)
- added L6: FB, kicad-libraries:R0603F, B.Cu at (145.3, 101.0)
- added R18: 5k1, kicad-libraries:R0603F, B.Cu at (140.7, 74.7)
- added R301: 82, kicad-libraries:R0402E, B.Cu at (164.2, 101.4)
- added R5: 5k1, kicad-libraries:R0603F, B.Cu at (145.0, 74.7)
- added R7: 1k, kicad-libraries:R0603F, B.Cu at (151.8, 84.3)
- added RP301: 82, kicad-libraries:4X0402, B.Cu at (156.0, 87.9)
- added RP302: 82, kicad-libraries:4X0402, B.Cu at (156.0, 90.7)
- added RP303: 82, kicad-libraries:4X0402, F.Cu at (155.8, 92.2)
- added RP304: 82, kicad-libraries:4X0402, B.Cu at (155.8, 95.1)
- added RP305: 82, kicad-libraries:4X0402, B.Cu at (162.5, 101.4)
- added RP306: 82, kicad-libraries:4X0402, F.Cu at (155.8, 97.9)
- added RP307: 82, kicad-libraries:4X0402, B.Cu at (152.9, 92.2)
- added RP308: 82, kicad-libraries:4X0402, B.Cu at (155.8, 97.9)
- added RP309: 1k, kicad-libraries:4X0402, F.Cu at (156.0, 82.2)
- added RP310: 82, kicad-libraries:4X0402, B.Cu at (156.0, 84.6)
- C10, C11: value 100nF -> DNP; footprint kicad-libraries:C0603 -> C0603
- C12, C13, C16, C18, C19, C20, C22, C23, C24, C25, C26, C27, C28, C30, C31, C32, C33, C34, C36, C37, C38, FB1, FB3: footprint kicad-libraries:C0603 -> C0603
- C14: value 1µF -> 1uF; footprint kicad-libraries:C0603 -> kicad-libraries:C0603F
- C15, C21, C29, C35, C39, L2: footprint kicad-libraries:C0805 -> C0805
- C17: footprint kicad-libraries:3528-21 -> 3528-21
- D1, D2, D3, D4, D5, D6: footprint kicad-libraries:D0603 -> D0603
- D11: footprint kicad-libraries:SOD-128 -> SOD-128
- FB4: footprint kicad-libraries:C0603 -> kicad-libraries:R0603F
- J1: value USB-MINI-B-SMD -> USB-C; footprint kicad-libraries:USB-MINI-B-SMD -> kicad-libraries:USB-C-2
- J2, J3, J4, J5: footprint kicad-libraries:DRILL_NP -> DRILL_NP
- J6, J8: value STACK-UP-LOW -> STACK-UP-HIGH; footprint kicad-libraries:BTB08-ACS-TOP -> BTB08-ACS-TOP
- J7, J9: footprint kicad-libraries:BTB08-ACS-BTM -> BTB08-ACS-BTM
- L1: footprint kicad-libraries:WE-CNSW-0603 -> WE-CNSW-0603
- P1: value CON-SENSOR -> Port A; footprint kicad-libraries:CON-SENSOR -> kicad-libraries:CON-SENSOR2
- P2: value CON-SENSOR -> Port B; footprint kicad-libraries:CON-SENSOR -> kicad-libraries:CON-SENSOR2
- P3: value CON-SENSOR -> Port C; footprint kicad-libraries:CON-SENSOR -> kicad-libraries:CON-SENSOR2
- P4: value CON-SENSOR -> Port D; footprint kicad-libraries:CON-SENSOR -> kicad-libraries:CON-SENSOR2
- P5, P6, P7: footprint kicad-libraries:TSTPT -> TSTPT
- Q1: footprint kicad-libraries:SOT23EBC -> kicad-libraries:SOT23GDS
- R10, R12: value 1k -> DNP; footprint kicad-libraries:R0603 -> R0603
- R11, R15, R16, R3, R4, R6, R8: footprint kicad-libraries:R0603 -> R0603
- R13, R9: value 10k -> DNP; footprint kicad-libraries:R0603 -> R0603
- R17: footprint kicad-libraries:R0603 -> R0603; moved to B.Cu
- RP3, RP4: footprint kicad-libraries:0603X4 -> 0603X4
- RP5, RP6: value 2k2 -> 82; footprint kicad-libraries:0603X4 -> kicad-libraries:4X0402
- RP7: value 2k2 -> 82; footprint kicad-libraries:0603X4 -> kicad-libraries:4X0402; moved to F.Cu
- RP8: footprint kicad-libraries:0603X4 -> kicad-libraries:4X0402
- RP9: value 10k -> 82; footprint kicad-libraries:0603X4 -> kicad-libraries:4X0402; moved to F.Cu
- SW1, SW2: footprint kicad-libraries:TACT-SWITCH -> TACT-SWITCH
- U1: value AT91SAM3SXC -> SAM4S4CA; footprint kicad-libraries:LQFP100 -> LQFP100
- U13: value RT9701XB -> STMPS2171STR; footprint kicad-libraries:SOT23-5 -> kicad-libraries:SOT23-5L
- U2: footprint kicad-libraries:SOT563-SPEC -> SOT563-SPEC
- U3: value PCA9518PW -> TPS22975; footprint kicad-libraries:TSSOP20 -> kicad-libraries:WSON8-2x2
- U4: value CM1293A -> AP7333-33SRG; footprint kicad-libraries:SC-74 -> kicad-libraries:SOT23-3
- X1: footprint kicad-libraries:CRYSTAL_3225 -> CRYSTAL_3225
- moved G*** 27.5 mm to (130.0, 78.0)
- moved RP5 19.4 mm to (135.1, 102.4), turned to 0 degrees
- moved U4 17.5 mm to (145.0, 90.8)
- moved RP7 17.0 mm to (138.9, 102.4), turned to 180 degrees
- moved U3 13.2 mm to (147.6, 85.5)
- moved C14 11.2 mm to (149.7, 85.3), turned to 270 degrees
- moved RP9 10.8 mm to (154.9, 102.5)
- moved RP6 7.64 mm to (151.1, 102.4), turned to 0 degrees
- moved R17 7.41 mm to (132.6, 102.5)
- moved R8 6.69 mm to (134.8, 75.6)
- moved D11 6.69 mm to (137.8, 73.3)
- moved Q1 6.69 mm to (131.8, 74.6)
- moved R11 6.69 mm to (134.8, 74.3)
- moved R6 6.69 mm to (134.8, 76.9)
- moved C36 6.52 mm to (134.1, 81.2), turned to 180 degrees
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Connections:
- net Net-(FB3-Pad1) renamed PGND
- C14 pad 1: GND -> VSTACK
- C14 pad 2: 3V3 -> GND
- C39 pad 1: VPP -> VCC
- D14 pad 2: VPP -> VCC
- FB4 pad 1: VSTACK -> Net-(FB4-Pad1)
- FB4 pad 2: Net-(FB4-Pad2) -> VSTACK
- J1 pad 5: GND -> Net-(J1-Pad5)
- J1 pad 6: Net-(FB2-Pad2) -> USB_GND
- J6 pad 1: STACK-SPI-MISO -> Net-(J6-Pad1)
- J6 pad 10: STACK-SELECT-02 -> Net-(J6-Pad10)
- J6 pad 11: STACK-SYNC/JTAG-TCK -> Net-(J6-Pad11)
- J6 pad 12: STACK-SELECT-03 -> Net-(J6-Pad12)
- J6 pad 13: STACK-SER-RXD -> Net-(J6-Pad13)
- J6 pad 14: STACK-SELECT-04 -> Net-(J6-Pad14)
- J6 pad 15: STACK-SER-TXD -> Net-(J6-Pad15)
- J6 pad 16: STACK-SELECT-05 -> Net-(J6-Pad16)
- J6 pad 17: STACK-SER-SCK -> Net-(J6-Pad17)
- J6 pad 18: STACK-SELECT-06 -> Net-(J6-Pad18)
- J6 pad 19: STACK-EX-0-GP00 -> Net-(J6-Pad19)
- J6 pad 2: STACK-I2C-SDA/JTAG-TDI -> Net-(J6-Pad2)
- J6 pad 20: STACK-SELECT-07 -> Net-(J6-Pad20)
- J6 pad 21: STACK-EX-0-GP01 -> Net-(J6-Pad21)
- J6 pad 22: STACK-SELECT-EX-00 -> Net-(J6-Pad22)
- J6 pad 23: STACK-EX-0-GP02 -> Net-(J6-Pad23)
- J6 pad 24: STACK-SELECT-EX-01 -> Net-(J6-Pad24)
- J6 pad 25: STACK-EX-1-GP00 -> Net-(J6-Pad25)
- J6 pad 26: STACK-SER2-RXD -> Net-(J6-Pad26)
- J6 pad 27: STACK-EX-1-GP01 -> Net-(J6-Pad27)
- J6 pad 28: STACK-SER2-TXD -> Net-(J6-Pad28)
- J6 pad 29: STACK-EX-1-GP02 -> Net-(J6-Pad29)
- J6 pad 3: STACK-SPI-MOSI -> Net-(J6-Pad3)
- J6 pad 30: STACK-SER2-RTS -> Net-(J6-Pad30)
- J6 pad 4: STACK-I2C-SCL/JTAG-TDO -> Net-(J6-Pad4)
- J6 pad 5: STACK-SPI-SCLK -> Net-(J6-Pad5)
- J6 pad 6: STACK-SELECT-00 -> Net-(J6-Pad6)
- J6 pad 8: STACK-SELECT-01 -> Net-(J6-Pad8)
- J6 pad 9: STACK-HIGH/JTAG-TMS -> Net-(J6-Pad9)
- J7 pad 1: STACK-SPI-MISO -> Net-(J6-Pad1)
- J7 pad 10: STACK-SELECT-01 -> Net-(J6-Pad8)
- J7 pad 11: STACK-SYNC/JTAG-TCK -> Net-(J6-Pad11)
- J7 pad 12: STACK-SELECT-02 -> Net-(J6-Pad10)
- J7 pad 13: STACK-SER-RXD -> Net-(J6-Pad13)
- J7 pad 14: STACK-SELECT-03 -> Net-(J6-Pad12)
- J7 pad 15: STACK-SER-TXD -> Net-(J6-Pad15)
- J7 pad 16: STACK-SELECT-04 -> Net-(J6-Pad14)
- J7 pad 17: STACK-SER-SCK -> Net-(J6-Pad17)
- J7 pad 18: STACK-SELECT-05 -> Net-(J6-Pad16)
- J7 pad 19: STACK-EX-0-GP00 -> Net-(J6-Pad19)
- J7 pad 2: STACK-I2C-SDA/JTAG-TDI -> Net-(J6-Pad2)
- J7 pad 20: STACK-SELECT-06 -> Net-(J6-Pad18)
- J7 pad 21: STACK-EX-0-GP01 -> Net-(J6-Pad21)
- J7 pad 22: STACK-SELECT-EX-00 -> Net-(J6-Pad22)
- J7 pad 23: STACK-EX-0-GP02 -> Net-(J6-Pad23)
- J7 pad 24: STACK-SELECT-EX-01 -> Net-(J6-Pad24)
- J7 pad 25: STACK-EX-1-GP00 -> Net-(J6-Pad25)
- J7 pad 26: STACK-SER2-RXD -> Net-(J6-Pad26)
- J7 pad 27: STACK-EX-1-GP01 -> Net-(J6-Pad27)
- J7 pad 28: STACK-SER2-TXD -> Net-(J6-Pad28)
- J7 pad 29: STACK-EX-1-GP02 -> Net-(J6-Pad29)
- J7 pad 3: STACK-SPI-MOSI -> Net-(J6-Pad3)
- J7 pad 30: STACK-SER2-RTS -> Net-(J6-Pad30)
- J7 pad 4: STACK-I2C-SCL/JTAG-TDO -> Net-(J6-Pad4)
- J7 pad 5: STACK-SPI-SCLK -> Net-(J6-Pad5)
- J7 pad 6: STACK-SPI-SELECT -> Net-(J7-Pad6)
- J7 pad 8: STACK-SELECT-00 -> Net-(J6-Pad6)
- J8 pad 22: Net-(FB4-Pad2) -> Net-(FB4-Pad1)
- J8 pad 24: Net-(FB4-Pad2) -> Net-(FB4-Pad1)
- J8 pad 26: Net-(FB4-Pad2) -> Net-(FB4-Pad1)
- J8 pad 28: VPP -> VCC
- J9 pad 22: Net-(FB4-Pad2) -> Net-(FB4-Pad1)
- J9 pad 24: Net-(FB4-Pad2) -> Net-(FB4-Pad1)
- J9 pad 26: Net-(FB4-Pad2) -> Net-(FB4-Pad1)
- J9 pad 28: VPP -> VCC
- P1 pad 1: VSTACK -> 5VBricklet
- P1 pad 2: GND -> GNDD1
- P1 pad 3: 3V3 -> 3,3VBricklet
- P1 pad 4: Net-(P1-Pad4) -> Net-(CP1-Pad4)
- P1 pad 5: Net-(P1-Pad5) -> Net-(CP1-Pad3)
- P1 pad 6: BRICKLET-SEL-0 -> Net-(CP1-Pad2)
- P1 pad 7: BRICKLET-IO0_0/AD0 -> Net-(P1-Pad7)
- P1 pad EP: GND -> GNDD1
- P2 pad 1: VSTACK -> 5VBricklet
- P2 pad 2: GND -> GNDD1
- P2 pad 3: 3V3 -> 3,3VBricklet
- P2 pad 4: Net-(P2-Pad4) -> Net-(CP2-Pad4)
- P2 pad 5: Net-(P2-Pad5) -> Net-(CP2-Pad3)
- P2 pad 6: BRICKLET-SEL-1 -> Net-(CP2-Pad2)
- P2 pad 7: BRICKLET-IO1_0/AD1 -> Net-(P2-Pad7)
- P2 pad EP: GND -> GNDD1
- P3 pad 1: VSTACK -> 5VBricklet
- P3 pad 2: GND -> GNDD1
- P3 pad 3: 3V3 -> 3,3VBricklet
- P3 pad 4: Net-(P3-Pad4) -> Net-(CP3-Pad4)
- P3 pad 5: Net-(P3-Pad5) -> Net-(CP3-Pad3)
- P3 pad 6: BRICKLET-SEL-2 -> Net-(CP3-Pad2)
- P3 pad 7: BRICKLET-IO2_0/AD2 -> Net-(P3-Pad7)
- P3 pad EP: GND -> GNDD1
- P4 pad 1: VSTACK -> 5VBricklet
- P4 pad 2: GND -> GNDD1
- P4 pad 3: 3V3 -> 3,3VBricklet
- P4 pad 4: Net-(P4-Pad4) -> Net-(CP4-Pad4)
- P4 pad 5: Net-(P4-Pad5) -> Net-(CP4-Pad3)
- P4 pad 6: BRICKLET-SEL-3 -> Net-(CP4-Pad2)
- P4 pad 7: BRICKLET-IO3_0/AD3 -> Net-(P4-Pad7)
- P4 pad EP: GND -> GNDD1
- R8 pad 2: Net-(Q1-Pad2) -> Net-(Q1-PadG)
- RP5 pad 1: 3V3 -> Port-A-MISO
- RP5 pad 2: 3V3 -> Port-A-MOSI
- RP5 pad 3: 3V3 -> Port-A-CLK
- RP5 pad 4: 3V3 -> Port-A-CS
- RP5 pad 5: BRICKLET-I2C-SDA -> Net-(CP1-Pad4)
- RP5 pad 6: Net-(RP5-Pad6) -> Net-(CP1-Pad3)
- RP5 pad 7: Net-(RP5-Pad7) -> Net-(CP1-Pad2)
- RP5 pad 8: BRICKLET-I2C-SCL -> Net-(P1-Pad7)
- RP6 pad 1: 3V3 -> Port-B-MISO
- RP6 pad 2: 3V3 -> Port-B-MOSI
- RP6 pad 3: 3V3 -> Port-B-CLK
- RP6 pad 4: 3V3 -> Port-B-CS
- RP6 pad 5: Net-(P3-Pad5) -> Net-(CP2-Pad4)
- RP6 pad 6: Net-(P3-Pad4) -> Net-(CP2-Pad3)
- RP6 pad 7: Net-(P1-Pad5) -> Net-(CP2-Pad2)
- RP6 pad 8: Net-(P1-Pad4) -> Net-(P2-Pad7)
- RP7 pad 1: 3V3 -> Port-C-MISO
- RP7 pad 2: 3V3 -> Port-C-MOSI
- RP7 pad 3: 3V3 -> Port-C-CLK
- RP7 pad 4: 3V3 -> Port-C-CS
- RP7 pad 5: Net-(P4-Pad5) -> Net-(CP3-Pad4)
- RP7 pad 6: Net-(P4-Pad4) -> Net-(CP3-Pad3)
- RP7 pad 7: Net-(P2-Pad5) -> Net-(CP3-Pad2)
- RP7 pad 8: Net-(P2-Pad4) -> Net-(P3-Pad7)
- RP8 pad 1: STACK-I2C-SCL/JTAG-TDO -> Net-(J6-Pad4)
- RP8 pad 4: STACK-I2C-SDA/JTAG-TDI -> Net-(J6-Pad2)
- RP9 pad 1: 3V3 -> Port-D-MISO
- RP9 pad 2: 3V3 -> Port-D-MOSI
- RP9 pad 3: 3V3 -> Port-D-CLK
- RP9 pad 4: 3V3 -> Port-D-CS
- RP9 pad 5: Net-(RP9-Pad5) -> Net-(CP4-Pad4)
- RP9 pad 6: Net-(RP9-Pad6) -> Net-(CP4-Pad3)
- RP9 pad 7: Net-(RP9-Pad7) -> Net-(CP4-Pad2)
- RP9 pad 8: Net-(RP9-Pad8) -> Net-(P4-Pad7)
- U1 pad 21: BRICKLET-IO1_0/AD1 -> Port-B-CS
- U1 pad 23: BRICKLET-IO0_0/AD0 -> Port-A-CS
- U1 pad 25: BRICKLET-IO0_2/PWM0 -> Port-A-MOSI
- U1 pad 29: BRICKLET-IO3_3 -> Port-D-MISO
- U1 pad 31: Net-(RP1-Pad4) -> STACK-SPI-SCLK
- U1 pad 32: BRICKLET-IO2_3 -> Port-C-MISO
- U1 pad 33: Net-(RP1-Pad3) -> STACK-SPI-MOSI
- U1 pad 35: BRICKLET-IO1_3 -> Port-B-MISO
- U1 pad 37: BRICKLET-IO0_3 -> Port-A-MISO
- U1 pad 38: BRICKLET-IO0_1 -> Port-A-CLK
- U1 pad 39: BRICKLET-IO1_1 -> Port-B-CLK
- U1 pad 4: BRICKLET-IO2_0/AD2 -> Port-C-CS
- U1 pad 40: BRICKLET-IO3_2/PWM3 -> Port-D-MOSI
- U1 pad 41: Net-(RP1-Pad2) -> STACK-SPI-MISO
- U1 pad 42: Net-(RP1-Pad1) -> STACK-SPI-SELECT
- U1 pad 43: BRICKLET-IO2_2/PWM2 -> Port-C-MOSI
- U1 pad 47: BRICKLET-IO1_2/PWM1 -> Port-B-MOSI
- U1 pad 49: Net-(U1-Pad49) -> Port-D-CS
- U1 pad 52: Net-(RP2-Pad2) -> STACK-SER-TXD
- U1 pad 53: Net-(RP2-Pad1) -> STACK-SER-RXD
- U1 pad 55: BRICKLET-I2C-SCL -> Port-D-CLK
- U1 pad 57: STACK-EX-0-GP02 -> STACK-EX-1-GP02
- U1 pad 58: BRICKLET-SEL-0 -> STACK-EX-0-GP02
- U1 pad 59: Net-(R1-Pad2) -> STACK-SELECT-EX-01
- U1 pad 6: BRICKLET-IO3_0/AD3 -> Net-(U1-Pad6)
- U1 pad 62: BRICKLET-SEL-1 -> Net-(U1-Pad62)
- U1 pad 63: Net-(R2-Pad2) -> STACK-SELECT-EX-00
- U1 pad 64: STACK-EX-1-GP01 -> STACK-EX-1-GP00
- U1 pad 65: BRICKLET-SEL-2 -> Net-(U1-Pad65)
- U1 pad 66: BRICKLET-I2C-SDA -> STACK-EX-1-GP01
- U1 pad 67: Net-(RP2-Pad3) -> STACK-SER-SCK
- U1 pad 68: BRICKLET-SEL-3 -> Net-(U1-Pad68)
- U1 pad 71: Net-(U1-Pad71) -> GND
- U1 pad 72: STACK-EX-1-GP00 -> Bricklet_Enable
- U1 pad 81: STACK-EX-1-GP02 -> Net-(U1-Pad81)
- U1 pad 93: BRICKLET-IO2_1/DA0 -> Port-C-CLK
- U1 pad 99: BRICKLET-IO3_1/DA1 -> Net-(U1-Pad99)
- U13 pad 1: VPP -> VCC
- U13 pad 3: 3V3 -> Net-(U13-Pad3)
- U13 pad 5: VPP -> 3V3
- U2 pad 2: GND -> USB_GND
- U3 pad 1: Net-(RP9-Pad5) -> VSTACK
- U3 pad 2: Net-(RP9-Pad6) -> VSTACK
- U3 pad 3: BRICKLET-I2C-SCL -> Bricklet_Enable
- U3 pad 4: BRICKLET-I2C-SDA -> VSTACK
- U3 pad 5: Net-(P2-Pad4) -> GND
- U3 pad 6: Net-(P2-Pad5) -> Net-(C40-Pad1)
- U3 pad 7: BRICKLET-SEL-1 -> Net-(C41-Pad2)
- U3 pad 8: Net-(P4-Pad4) -> Net-(C41-Pad2)
- U4 pad 1: BRICKLET-IO0_0/AD0 -> GND
- U4 pad 2: GND -> Net-(C43-Pad2)
- U4 pad 3: Net-(P1-Pad4) -> Net-(C41-Pad2)
Routing:
- net GND: track 424.3 -> 215.6 mm, vias 71 -> 82
- net 3V3: track 307.1 -> 107.6 mm, vias 32 -> 22
- net BRICKLET-IO3_1/DA1: track 33.2 -> 0.00 mm
- net BRICKLET-IO2_1/DA0: track 30.5 -> 0.00 mm, vias 2 -> 0
- net BRICKLET-IO3_0/AD3: track 30.0 -> 0.00 mm
- net USB_GND: track 0.00 -> 29.7 mm, vias 0 -> 7
- net BRICKLET-SEL-2: track 29.3 -> 0.00 mm, vias 2 -> 0
- net BRICKLET-IO3_3: track 28.6 -> 0.00 mm, vias 2 -> 0
- net BRICKLET-SEL-3: track 28.6 -> 0.00 mm, vias 3 -> 0
- net VPP: track 27.4 -> 0.00 mm, vias 3 -> 0
- net BRICKLET-SEL-0: track 26.4 -> 0.00 mm, vias 2 -> 0
- net BRICKLET-IO2_0/AD2: track 25.1 -> 0.00 mm, vias 2 -> 0
- net BRICKLET-IO1_0/AD1: track 24.9 -> 0.00 mm, vias 2 -> 0
- net Net-(RP1-Pad4): track 24.2 -> 0.00 mm, vias 2 -> 0
- net BRICKLET-SEL-1: track 23.9 -> 0.00 mm, vias 2 -> 0
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- added copper zone on VCC, net 3,3VBricklet
- added copper zone on B.Cu, net 5VBricklet
- added copper zone on B.Cu, net GNDD1
- added copper zone on F.Cu, net GNDD1
- added copper zone on GND, net GNDD1
- added copper zone on B.Cu, net Net-(C41-Pad2)
- added copper zone on B.Cu, net VSTACK
- removed copper zone on B.Cu, net 3V3
- removed copper zone on F.Cu, net 3V3
Other:
- net class Default: clearance 0.14986 -> 0.149; trace_width 0.14986 -> 0.15; via_dia 0.70104 -> 0.7; via_drill 0.24892 -> 0.4
- rule trace_clearance: 0.14986 -> 0.149
- rule via_min_drill: 0.24874 -> 0.25
- rule via_min_size: 0.6986 -> 0.4
- board text added: "Copyright Tinkerforge GmbH 2020. This documentation describes Open Hardware and is licensed under the CERN OHL v. 1.1. You may redistribute and modify this documentation under the terms of the CERN OHL v.1.1. (http://ohwr.org/cernohl). This documentation is distributed WITHOUT ANY EXPRESS OR IMPLIED WARRANTY, INCLUDING OF MERCHANTABILITY, SATISFACTORY QUALITY AND FITNESS FOR A PARTICULAR PURPOSE.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"
- board text added: "Master 3.1"
- board text removed: "Copyright Tinkerforge GmbH 2017. This documentation describes Open Hardware and is licensed under the CERN OHL v. 1.1. You may redistribute and modify this documentation under the terms of the CERN OHL v.1.1. (http://ohwr.org/cernohl). This documentation is distributed WITHOUT ANY EXPRESS OR IMPLIED WARRANTY, INCLUDING OF MERCHANTABILITY, SATISFACTORY QUALITY AND FITNESS FOR A PARTICULAR PURPOSE.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"
- board text removed: "Master 2.1"
